Commit message: added realsense xacro

File: rotors_description/urdf/component_snippets.xacro (robot description, xacro)
@@ -49,5 +49,5 @@
             <xacro:insert_block name="geometry" />
           </geometry>
-          <material name="red" />
+          <material name="Blue" />
         </visual>
       </xacro:if>
@@ -665,5 +665,5 @@
   </xacro:macro>
   <!-- VI-Sensor Macro -->
-  <xacro:macro name="vi_sensor_macro" params="namespace parent_link enable_cameras enable_depth enable_ground_truth *origin">
+  <xacro:macro name="vi_sensor_macro" params="namespace parent_link enable_cameras enable_depth enable_ground_truth *origin enable_visual">
     <!-- Vi Sensor Link -->
     <link name="${namespace}/vi_sensor_link">
@@ -674,10 +674,12 @@
         </geometry>
       </collision>
-      <visual>
-        <origin xyz="0 0 0" rpy="0 0 0" />
-        <geometry>
-          <mesh filename="package://rotors_description/meshes/vi_sensor.dae" scale="1 1 1" />
-        </geometry>
-      </visual>
+      <xacro:if value="${enable_visual}">
+        <visual>
+          <origin xyz="0 0 0" rpy="0 0 0" />
+          <geometry>
+            <mesh filename="package://rotors_description/meshes/vi_sensor.dae" scale="1 1 1" />
+          </geometry>
+        </visual>
+      </xacro:if>
       <inertial>
         <mass value="0.13" />

File: rotors_description/urdf/multirotor_base.xacro (robot description, xacro)
@@ -60,5 +60,5 @@
         <origin xyz="0 0 0" rpy="0 0 0" />
         <geometry>
-          <box size="${body_width} ${body_width} ${body_height}" /> <!-- [m] [m] [m] -->
+          <box size="${body_width} ${body_width} ${body_height}" /> <!-- [m] [m] [m] JDS: original "${body_width} ${body_width} ${body_height}" -->
         </geometry>
       </collision>

File: rotors_description/urdf/tyrion.xacro (robot description, xacro)
@@ -24,8 +24,8 @@
   <xacro:property name="mass" value="1.5" /> <!-- [kg] -->
   <xacro:property name="body_width" value="0.1" /> <!-- [m] -->
-  <xacro:property name="body_height" value="0.5" /> <!-- [m] JDS: original value="0.16"-->
-  <xacro:property name="mass_rotor" value="0.005" /> <!-- [kg] -->
-  <xacro:property name="arm_length" value="0.215" /> <!-- [m] -->
-  <xacro:property name="rotor_offset_top" value="0.1" /> <!-- [m] JDS: prop height?: original "0.037"-->
+  <xacro:property name="body_height" value="0.16" /> <!-- [m] JDS: original value="0.16"-->
+  <xacro:property name="mass_rotor" value="0.0054" /> <!-- [kg] JDS: original value="0.005" -->
+  <xacro:property name="arm_length" value="0.281" /> <!-- [m] JDS: original value="0.215" -->
+  <xacro:property name="rotor_offset_top" value="0.061" /> <!-- [m] JDS: prop height?: original "0.037"-->
   <xacro:property name="radius_rotor" value="0.1" /> <!-- [m] -->
   <xacro:property name="motor_constant" value="8.54858e-06" /> <!-- [kg m/s^2] -->

Commit message: Starting to add cameras (need tf)

File: rotors_description/urdf/component_snippets.xacro (robot description, xacro)
@@ -665,5 +665,5 @@
   </xacro:macro>
   <!-- VI-Sensor Macro -->
-  <xacro:macro name="vi_sensor_macro" params="namespace parent_link enable_cameras enable_depth enable_ground_truth *origin enable_visual">
+  <xacro:macro name="vi_sensor_macro" params="namespace parent_link enable_cameras enable_depth enable_ground_truth *origin">
     <!-- Vi Sensor Link -->
     <link name="${namespace}/vi_sensor_link">
@@ -674,12 +674,10 @@
         </geometry>
       </collision>
-      <xacro:if value="${enable_visual}">
-        <visual>
-          <origin xyz="0 0 0" rpy="0 0 0" />
-          <geometry>
-            <mesh filename="package://rotors_description/meshes/vi_sensor.dae" scale="1 1 1" />
-          </geometry>
-        </visual>
-      </xacro:if>
+      <visual>
+        <origin xyz="0 0 0" rpy="0 0 0" />
+        <geometry>
+          <mesh filename="package://rotors_description/meshes/vi_sensor.dae" scale="1 1 1" />
+        </geometry>
+      </visual>
       <inertial>
         <mass value="0.13" />

Commit message: Adding realsense Cameras

File: rotors_description/urdf/component_snippets.xacro (robot description, xacro)
@@ -49,5 +49,7 @@
             <xacro:insert_block name="geometry" />
           </geometry>
-          <material name="Blue" />
+          <material name="aluminum">
+            <color rgba="0.5 0.5 0.5 1"/>
+          </material>
         </visual>
       </xacro:if>

Commit message: tyrion working with waypoint

File: rotors_description/urdf/component_snippets.xacro (robot description, xacro)
@@ -683,5 +683,5 @@
       </visual>
       <inertial>
-        <mass value="0.13" />
+        <mass value="0.013" />
         <origin xyz="0 0 0" rpy="0 0 0" />
         <inertia ixx="1e-6" ixy="0" ixz="0" iyy="1e-6" iyz="0" izz="1e-6" />
@@ -769,5 +769,5 @@
       parent_link="${parent_link}"
       imu_topic="ground_truth/imu"
-      mass_imu_sensor="0.00001"
+      mass_imu_sensor="0.001"
       gyroscope_noise_density="0.0"
       gyroscope_random_walk="0.0"
@@ -778,5 +778,5 @@
       accelerometer_bias_correlation_time="300.0"
       accelerometer_turn_on_bias_sigma="0.0">
-      <inertia ixx="0.00001" ixy="0.0" ixz="0.0" iyy="0.00001" iyz="0.0" izz="0.00001" />
+      <inertia ixx="0.000001" ixy="0.0" ixz="0.0" iyy="0.000001" iyz="0.0" izz="0.000001" />
       <origin xyz="0 0 0" rpy="0 0 0" />
     </xacro:imu_plugin_macro>
@@ -819,5 +819,5 @@
       parent_link="${parent_link}"
       imu_topic="imu"
-      mass_imu_sensor="0.015"
+      mass_imu_sensor="0.00015"
       gyroscope_noise_density="0.0003394"
       gyroscope_random_walk="0.000038785"
@@ -856,5 +856,5 @@
       parent_link="${parent_link}"
       magnetometer_topic="magnetic_field"
-      mass_magnetometer_sensor="0.015"
+      mass_magnetometer_sensor="0.0015"
       ref_mag_north="0.000021493"
       ref_mag_east="0.000000815"
@@ -872,5 +872,5 @@
       parent_link="${parent_link}"
       pressure_topic="air_pressure"
-      mass_pressure_sensor="0.015"
+      mass_pressure_sensor="0.0015"
       reference_altitude="500.0"
       pressure_variance="0.0">

File: rotors_description/urdf/multirotor_base.xacro (robot description, xacro)
@@ -60,5 +60,5 @@
         <origin xyz="0 0 0" rpy="0 0 0" />
         <geometry>
-          <box size="${body_width} ${body_width} ${body_height}" /> <!-- [m] [m] [m] JDS: original "${body_width} ${body_width} ${body_height}" -->
+          <box size="0.5 0.5 0.35" /> <!-- [m] [m] [m] JDS: original "${body_width} ${body_width} ${body_height}" -->
         </geometry>
       </collision>

Commit message: adding props and testint joystick

File: rotors_description/urdf/component_snippets.xacro (robot description, xacro)
@@ -662,4 +662,71 @@
           <distortionT1>0.0</distortionT1>
           <distortionT2>0.0</distortionT2>
+        </plugin>
+      </sensor>
+    </gazebo>
+  </xacro:macro>
+  <!-- Macro to add a Lidar sensor. -->
+  <xacro:macro name="hokuyo_macro"
+    params="namespace parent_link ">
+    <!-- Hokuyo Laser joint -->
+    <joint name="hokuyo_joint" type="fixed">
+      <axis xyz="0 1 0" />
+      <origin xyz="0 0 1" rpy="0 0 0"/>
+      <parent link="${parent_link}" />
+      <child link="${namespace}/hokuyo_link" />
+    </joint>
+    <!-- Hokuyo Laser link-->
+    <link name="hokuyo_link">
+      <collision>
+        <origin xyz="0 0 0" rpy="0 0 0"/>
+        <geometry>
+          <box size="0.1 0.1 0.1"/>
+        </geometry>
+      </collision>
+      <visual>
+        <origin xyz="0 0 0" rpy="0 0 0"/>
+        <geometry>
+          <mesh filename="package://rrbot_description/meshes/hokuyo.dae"/>
+        </geometry>
+      </visual>
+      <inertial>
+        <mass value="1e-5" />
+        <origin xyz="0 0 0" rpy="0 0 0"/>
+        <inertia ixx="1e-6" ixy="0" ixz="0" iyy="1e-6" iyz="0" izz="1e-6" />
+      </inertial>
+    </link>
+    <!-- hokuyo -->
+    <gazebo reference="hokuyo_link">
+      <sensor type="gpu_ray" name="head_hokuyo_sensor">
+        <pose>0 0 0 0 0 0</pose>
+        <visualize>false</visualize>
+        <update_rate>40</update_rate>
+        <ray>
+          <scan>
+            <horizontal>
+              <samples>720</samples>
+              <resolution>1</resolution>
+              <min_angle>-1.570796</min_angle>
+              <max_angle>1.570796</max_angle>
+            </horizontal>
+          </scan>
+          <range>
+            <min>0.10</min>
+            <max>30.0</max>
+            <resolution>0.01</resolution>
+          </range>
+          <noise>
+            <type>gaussian</type>
+            <!-- Noise parameters based on published spec for Hokuyo laser
+                achieving "+-30mm" accuracy at range < 10m.  A mean of 0.0m and
+                stddev of 0.01m will put 99.7% of samples within 0.03m of the true
+                reading. -->
+            <mean>0.0</mean>
+            <stddev>0.01</stddev>
+          </noise>
+        </ray>
+        <plugin name="${namespace}_camera_{camera_suffix}" filename="libgazebo_ros_gpu_laser.so">
+          <topicName>/rrbot/laser/scan</topicName>
+          <frameName>hokuyo_link</frameName>
         </plugin>
       </sensor>

File: rotors_description/urdf/tyrion.xacro (robot description, xacro)
@@ -27,5 +27,5 @@
   <xacro:property name="mass_rotor" value="0.0054" /> <!-- [kg] JDS: original value="0.005" -->
   <xacro:property name="arm_length" value="0.281" /> <!-- [m] JDS: original value="0.215" -->
-  <xacro:property name="rotor_offset_top" value="0.061" /> <!-- [m] JDS: prop height?: original "0.037"-->
+  <xacro:property name="rotor_offset_top" value="0.05" /> <!-- [m] JDS: prop height?: original "0.037"-->
   <xacro:property name="radius_rotor" value="0.1" /> <!-- [m] -->
   <xacro:property name="motor_constant" value="8.54858e-06" /> <!-- [kg m/s^2] -->
