Commit message: workind xacro in RVIZ

File: rotors_description/urdf/multirotor_base.xacro (robot description, xacro)
@@ -49,10 +49,12 @@
         <origin xyz="0 0 0" rpy="0 0 0" />
         <geometry>
-          <xacro:if value="${use_mesh_file}">
+        <!-- JDS change to force mesh to check why not showing in rviz-->
+          <mesh filename="package://rotors_description/meshes/tyrion_nosensors.dae" scale="1 1 1" />
+          <!-- <xacro:if value="${use_mesh_file}">
             <mesh filename="${mesh_file}" scale="1 1 1" />
           </xacro:if>
           <xacro:unless value="${use_mesh_file}">
-            <box size="${body_width} ${body_width} ${body_height}"/> <!-- [m] [m] [m] -->
-          </xacro:unless>
+            <box size="${body_width} ${body_width} ${body_height}"/> [m] [m] [m]
+          </xacro:unless> -->
         </geometry>
       </visual>

File: rotors_description/urdf/tyrion.xacro (robot description, xacro)
@@ -21,5 +21,5 @@
   <xacro:property name="rotor_velocity_slowdown_sim" value="10" />
   <xacro:property name="use_mesh_file" value="true" />
-  <xacro:property name="mesh_file" value="package://rotors_description/meshes/tyrion.dae" />
+  <xacro:property name="mesh_file" value="package://rotors_description/meshes/tyrion_nosensors.dae" />
   <xacro:property name="mass" value="1.5" /> <!-- [kg] -->
   <xacro:property name="body_width" value="0.1" /> <!-- [m] -->
@@ -75,5 +75,5 @@
     rotor_drag_coefficient="${rotor_drag_coefficient}"
     rolling_moment_coefficient="${rolling_moment_coefficient}"
-    color="Red"
+    color="Grey"
     use_own_mesh="false"
     mesh="">
@@ -96,5 +96,5 @@
     rotor_drag_coefficient="${rotor_drag_coefficient}"
     rolling_moment_coefficient="${rolling_moment_coefficient}"
-    color="Blue"
+    color="Black"
     use_own_mesh="false"
     mesh="">
@@ -116,5 +116,5 @@
     rotor_drag_coefficient="${rotor_drag_coefficient}"
     rolling_moment_coefficient="${rolling_moment_coefficient}"
-    color="Blue"
+    color="Black"
     use_own_mesh="false"
     mesh="">
@@ -136,5 +136,5 @@
     rotor_drag_coefficient="${rotor_drag_coefficient}"
     rolling_moment_coefficient="${rolling_moment_coefficient}"
-    color="Blue"
+    color="Black"
     use_own_mesh="false"
     mesh="">
@@ -157,5 +157,5 @@
     rotor_drag_coefficient="${rotor_drag_coefficient}"
     rolling_moment_coefficient="${rolling_moment_coefficient}"
-    color="Blue"
+    color="Black"
     use_own_mesh="false"
     mesh="">
@@ -178,5 +178,5 @@
     rotor_drag_coefficient="${rotor_drag_coefficient}"
     rolling_moment_coefficient="${rolling_moment_coefficient}"
-    color="Red"
+    color="Grey"
     use_own_mesh="false"
     mesh="">
